File: kicad/power.kicad_sch (KiCad schematic)
At the start: 97 parts, among them J1 USB_C_Receptacle_USB2.0_16P, J11 Balance, J2 NTC bead 10k B3435, J3 XT60-F pigtail 14AWG, Q1 AO4407A, Q2 80N03F, Q3 80N03F, SW1 Power, U13 BQ7791501, U4 AP64500SP-13, U5 CH224A, U7 BQ25798, U8 HT7550-1, U9 XC6206P332MR

Commit message: Re-lay out rev 2 around an Ovonic 450 pack on top of the board
The internal pack is now an Ovonic 3S 450 mAh XT30 pack sitting 2 mm
above the board over the low-power logic area, on an XT30 pigtail. The
board is 88.5 x 47 mm with 2 mm corner radii, for a box of about
93.5 x 52 x 24.6 mm whose face has no openings.

- IO S1-S6 are a 3 x 6 right-angle header out of the left end, beside
  M5/M6, replacing the recessed vertical block.
- BOOT is a side-push switch on the top edge behind a pinhole sized for
  a 2.5 mm hex key; RESET is removed, with RUN on a bottom test pad
  beside SWCLK/SWDIO/GND.
- The CHG LED is a side-view part on the top edge; the GPIO status LED
  is removed now that the WS2812B stick shows status.
- The pack NTC is removed (a fixed 10k holds the charger's TS at 25 C);
  the protector's on-board TH1 stays.
- Q1, F1 and the other warm parts moved out from under the pack, and the
  GPIO map was re-swapped for the new placement (I2C on I2C1).

Schematic review passes; PCB review passes every gate except unrouted.

Co-Authored-By: Claude Opus 5.5 <noreply@anthropic.com>
Parts:
- removed J2: NTC bead 10k B3435, Connector_Wire:SolderWire-0.1sqmm_1x02_P3.6mm_D0.4mm_OD1mm, symbol Connector_Generic:Conn_01x02
- added R81: 10k, Resistor_SMD:R_0402_1005Metric, symbol Device:R
- J3: value XT60-F pigtail 14AWG -> XT30 pigtail 16AWG; footprint Connector_Wire:SolderWire-2sqmm_1x02_P7.8mm_D2mm_OD3.9mm -> Connector_Wire:SolderWire-1.5sqmm_1x02_P6mm_D1.7mm_OD3mm
- LED1: footprint LED_SMD:LED_0805_2012Metric -> hexy:LED_Everlight_27-21_SideView; LCSC Part # C2297 -> C74270; MPN KT-0805G -> 27-21SYGC/S530-E3/TR8; Manufacturer Hubei KENTO Elec -> Everlight Elec
Connections:
- net GND: now also R81.2
- net at R34.2, R35.1, U7.16 (TS): now also R81.1
Other:
- note added: "CHARGE SAFETY WITHOUT FIRMWARE PROG: R31 + R78 (2 x 6.8 k = 13.6 k) select 3S (12.6 V) at 750 kHz. ILIM_HIZ: R32/R33 (100 k / 33 k from REGN) set 1.24 V, an input limit of about 0.30 A. Charge current stays near 0.2 A (about 0.45C of the 450 mAh pack) from 9 V (less from 5 V), even though the power-on charge-current default is 1 A. TS: R34/R35 with a fixed 10 k (R81, no pack NTC) hold TS at the 2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"
- note added: "MOTORS BYPASS THE CHARGER SYS VSYS (motors, 5 V buck) comes from the pack through F1 and Q1, not from CHG_SYS: the BQ25798 BATFET is rated 6 A continuous, below the motor peaks. CHG_SYS only carries its own caps. Charging works with the power switch off. LED1 (green, side view on the top edge, seen through a small hole in the wall) is lit while charging, no firmware needed."
- note added: "PACK PROTECTION (Ovonic 80C 3S 450 mAh, no protection board in the pack)"
- note removed: "CHARGE SAFETY WITHOUT FIRMWARE PROG: R31 13.7 k selects 3S (12.6 V) at 750 kHz. ILIM_HIZ: R32/R33 (100 k / 33 k from REGN) set 1.24 V, an input limit of about 0.30 A. Charge current stays near 0.22C of the 1000 mAh pack from 9 V (less from 5 V), even though the power-on charge-current default is 1 A. TS: R34/R35 with a 10 k B3435 bead on J2 (taped to the pack) give JEITA limits. /CE tied low: cha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"
- note removed: "MOTORS BYPASS THE CHARGER SYS VSYS (motors, 5 V buck) comes from the pack through F1 and Q1, not from CHG_SYS: the BQ25798 BATFET is rated 6 A continuous, below the motor peaks. CHG_SYS only carries its own caps. Charging works with the power switch off. LED1 (green) is lit while charging, no firmware needed."
- note removed: "PACK PROTECTION (Gens Ace 3S 1000 mAh, no protection board in the pack)"
Changed lines of the file:
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@@
 			)
 		)
-		(property "Footprint" "LED_SMD:LED_0805_2012Metric"
+		(property "Footprint" "hexy:LED_Everlight_27-21_SideView"
 			(at 237.49 78.74 0)
 			(hide yes)
@@
 			)
 		)
-		(property "MPN" "KT-0805G"
+		(property "MPN" "27-21SYGC/S530-E3/TR8"
 			(at 237.49 78.74 0)
 			(effects
@@
 			)
 		)
-		(property "Manufacturer" "Hubei KENTO Elec"
+		(property "Manufacturer" "Everlight Elec"
 			(at 237.49 78.74 0)
 			(effects
@@
 			)
 		)
-		(property "LCSC Part #" "C2297"
+		(property "LCSC Part #" "C74270"
 			(at 237.49 78.74 0)
 			(effects
@@
 	)
 	(symbol
-		(lib_id "Connector_Generic:Conn_01x02")
-		(at 175.26 116.84 0)
-		(mirror y)
-		(unit 1)
-		(exclude_from_sim no)
-		(in_bom yes)
-		(on_board yes)
-		(dnp no)
-		(property "Reference" "J2"
-			(at 168.91 116.84 0)
-			(show_name no)
-			(do_not_autoplace no)
-			(effects
-				(font
-					(size 1.27 1.27)
-				)
-			)
-		)
-		(property "Value" "NTC bead 10k B3435"
-			(at 167.64 119.38 0)
-			(show_name no)
-			(do_not_autoplace no)
-			(effects
-				(font
-					(size 1.27 1.27)
-				)
-			)
-		)
-		(property "Footprint" "Connector_Wire:SolderWire-0.1sqmm_1x02_P3.6mm_D0.4mm_OD1mm"
-			(at 175.26 116.84 0)
-			(hide yes)
-			(show_name no)
-			(do_not_autoplace no)
-			(effects
-				(font
-					(size 1.27 1.27)
-				)
-			)
-		)
-		(property "Datasheet" ""
-			(at 175.26 116.84 0)
-			(hide yes)
-			(show_name no)
-			(do_not_autoplace no)
-			(effects
-				(font
-					(size 1.27 1.27)
-				)
-			)
-		)
-		(property "Description" "Generic connector, single row, 01x02, script generated (kicad-library-utils/schlib/autogen/connector/)"
-			(at 175.26 116.84 0)
-			(hide yes)
-			(show_name no)
-			(do_not_autoplace no)
-			(effects
-				(font
-					(size 1.27 1.27)
-				)
-			)
-		)
-		(property "MPN" ""
-			(at 175.26 116.84 0)
-			(effects
-				(font
-					(size 1.27 1.27)
-				)
-				(hide yes)
-			)
-		)
-		(property "Manufacturer" ""
-			(at 175.26 116.84 0)
-			(effects
-				(font
-					(size 1.27 1.27)
-				)
-				(hide yes)
-			)
-		)
-		(pin "1"
-		)
-		(pin "2"
-		)
-		(instances
-			(project "thegoose"
-				(path "/72b1d502-e600-4337-8ef9-b222b53a12da/0021e6ae-34c0-486e-ac47-c8566b803df5"
-					(reference "J2")
-					(unit 1)
-				)
-			)
-		)
-	)
-	(symbol
 		(lib_id "power:GND")
-		(at 180.34 119.38 0)
+		(at 180.34 124.46 0)
 		(unit 1)
 		(exclude_from_sim no)
@@
 		(dnp no)
 		(property "Reference" "#PWR139"
-			(at 180.34 116.84 0)
+			(at 180.34 121.92 0)
 			(show_name no)
 			(do_not_autoplace no)
@@
 		)
 		(property "Value" "GND"
-			(at 180.34 123.19 0)
+			(at 180.34 128.27 0)
 			(show_name no)
 			(do_not_autoplace no)
@@
 		)
 		(property "Footprint" ""
-			(at 180.34 119.38 0)
+			(at 180.34 124.46 0)
 			(hide yes)
 			(show_name no)
@@
 		)
 		(property "Datasheet" ""
-			(at 180.34 119.38 0)
+			(at 180.34 124.46 0)
 			(hide yes)
 			(show_name no)
@@
 		)
 		(property "Description" "Power symbol creates a global label with name \"GND\" , ground"
-			(at 180.34 119.38 0)
+			(at 180.34 124.46 0)
 			(hide yes)
 			(show_name no)
@@
 			)
 		)
-		(property "Value" "XT60-F pigtail 14AWG"
+		(property "Value" "XT30 pigtail 16AWG"
 			(at 153.67 172.72 0)
 			(show_name no)
@@
 			)
 		)
-		(property "Footprint" "Connector_Wire:SolderWire-2sqmm_1x02_P7.8mm_D2mm_OD3.9mm"
+		(property "Footprint" "Connector_Wire:SolderWire-1.5sqmm_1x02_P6mm_D1.7mm_OD3mm"
 			(at 160.02 170.18 0)
 			(hide yes)
@@
 		)
 	)
-	(text "CHARGE SAFETY WITHOUT FIRMWARE\nPROG: R31 13.7 k selects 3S (12.6 V) at 750 kHz.\nILIM_HIZ: R32/R33 (100 k / 33 k from REGN) set 1.24 V, an input\nlimit of about 0.30 A. Charge current stays near 0.22C of the\n1000 mAh pack from 9 V (less from 5 V), even though the\npower-on charge-current default is 1 A.\nTS: R34/R35 with a 10 k B3435 bead on J2 (taped to the pack) give JEITA limits.\n/CE tied low: charging always on. /QON, D+/D- unused.\nNo ship FET: SDRV only has C36. BATP senses VBAT via R30.\nFirmware may raise the limits over I2C (GPIO12/13, /INT GPIO14)."
+	(text "CHARGE SAFETY WITHOUT FIRMWARE\nPROG: R31 + R78 (2 x 6.8 k = 13.6 k) select 3S (12.6 V) at 750 kHz.\nILIM_HIZ: R32/R33 (100 k / 33 k from REGN) set 1.24 V, an input\nlimit of about 0.30 A. Charge current stays near 0.2 A (about 0.45C of the\n450 mAh pack) from 9 V (less from 5 V), even though the\npower-on charge-current default is 1 A.\nTS: R34/R35 with a fixed 10 k (R81, no pack NTC) hold TS at the 25 C point (58.9 % of REGN): always the normal zone.\n/CE tied low: charging always on. /QON, D+/D- unused.\nNo ship FET: SDRV only has C36. BATP senses VBAT via R30.\nFirmware may raise the limits over I2C0 (SDA GPIO8, SCL GPIO17, /INT GPIO9)."
 		(exclude_from_sim no)
 		(at 271.78 45.72 0)
@@
 		)
 	)
-	(text "MOTORS BYPASS THE CHARGER SYS\nVSYS (motors, 5 V buck) comes from the pack through F1 and Q1,\nnot from CHG_SYS: the BQ25798 BATFET is rated 6 A continuous,\nbelow the motor peaks. CHG_SYS only carries its own caps.\nCharging works with the power switch off.\nLED1 (green) is lit while charging, no firmware needed."
+	(text "MOTORS BYPASS THE CHARGER SYS\nVSYS (motors, 5 V buck) comes from the pack through F1 and Q1,\nnot from CHG_SYS: the BQ25798 BATFET is rated 6 A continuous,\nbelow the motor peaks. CHG_SYS only carries its own caps.\nCharging works with the power switch off.\nLED1 (green, side view on the top edge, seen through a small hole in the wall)\nis lit while charging, no firmware needed."
 		(exclude_from_sim no)
 		(at 271.78 83.82 0)
@@
 		(at 162.56 250.19)
 	)
-	(text "PACK PROTECTION (Gens Ace 3S 1000 mAh, no protection board in the pack)"
+	(text "PACK PROTECTION (Ovonic 80C 3S 450 mAh, no protection board in the pack)"
 		(exclude_from_sim no)
 		(at 40 204 0)
@@
 		)
 	)
-	(text "BQ7791501 standalone 3S (datasheet Fig. 9-11): OV 4.25 V, UV 2.8 V; 2.5 mOhm shunt (R66||R67) -> OCD1 14 A, OCD2 24 A, SCD 48 A, OCC 8 A.\nCCFG, CTRC, CTRD, CBI to VSS (3 cells, no stack, balancing on); PRES high through R75 (no HIBERNATE); R76 100k = EEPROM OCD delays.\nGround: the pack's negative (BAT_N, J3 pin 1) -> shunt -> Q2 (DSG) -> Q3 (CHG) -> board GND (PACK-). Everything else runs on board GND.\nTH1 (0603 by the FETs) is the protector's TS; the charger's TS bead is J2. Balance lead J11: pin 1 cell 1-, pin 4 cell 3+."
+	(text "BQ7791501 standalone 3S (datasheet Fig. 9-11): OV 4.25 V, UV 2.8 V; 2.5 mOhm shunt (R66||R67) -> OCD1 14 A, OCD2 24 A, SCD 48 A, OCC 8 A.\nCCFG, CTRC, CTRD, CBI to VSS (3 cells, no stack, balancing on); PRES high through R75 (no HIBERNATE); R76 100k = EEPROM OCD delays.\nGround: the pack's negative (BAT_N, J3 pin 1) -> shunt -> Q2 (DSG) -> Q3 (CHG) -> board GND (PACK-). Everything else runs on board GND.\nTH1 (0603 by the FETs) is the protector's TS; the charger's TS has a fixed 10 k (R81) instead of a pack NTC. Balance lead J11: pin 1 cell 1-, pin 4 cell 3+."
 		(exclude_from_sim no)
 		(at 40 284 0)
@@
 		)
 	)
+	(symbol
+		(lib_id "Device:R")
+		(at 180.34 120.65 0)
+		(unit 1)
+		(exclude_from_sim no)
+		(in_bom yes)
+		(on_board yes)
+		(dnp no)
+		(property "Reference" "R81"
+			(at 177.8 119.38 0)
+			(show_name no)
+			(do_not_autoplace no)
+			(effects
+				(font
+					(size 1.27 1.27)
+				)
+				(justify right)
+			)
+		)
+		(property "Value" "10k"
+			(at 177.8 121.92 0)
+			(show_name no)
+			(do_not_autoplace no)
+			(effects
+				(font
+					(size 1.27 1.27)
+				)
+				(justify right)
+			)
+		)
+		(property "Footprint" "Resistor_SMD:R_0402_1005Metric"
+			(at 178.562 120.65 90)
+			(hide yes)
+			(show_name no)
+			(do_not_autoplace no)
+			(effects
+				(font
+					(size 1.27 1.27)
+				)
+			)
+		)
+		(property "Datasheet" ""
+			(at 180.34 120.65 0)
+			(hide yes)
+			(show_name no)
+			(do_not_autoplace no)
+			(effects
+				(font
+					(size 1.27 1.27)
+				)
+			)
+		)
+		(property "Description" "Resistor"
+			(at 180.34 120.65 0)
+			(hide yes)
+			(show_name no)
+			(do_not_autoplace no)
+			(effects
+				(font
+					(size 1.27 1.27)
+				)
+			)
+		)
+		(property "MPN" "0402WGF1002TCE"
+			(at 180.34 120.65 0)
+			(effects
+				(font
+					(size 1.27 1.27)
+				)
+				(hide yes)
+			)
+		)
+		(property "Manufacturer" "UNI-ROYAL"
+			(at 180.34 120.65 0)
+			(effects
+				(font
+					(size 1.27 1.27)
+				)
+				(hide yes)
+			)
+		)
+		(property "LCSC Part #" "C25744"
+			(at 180.34 120.65 0)
+			(effects
+				(font
+					(size 1.27 1.27)
+				)
+				(hide yes)
+			)
+		)
+		(pin "1"
+		)
+		(pin "2"
+		)
+		(instances
+			(project "thegoose"
+				(path "/72b1d502-e600-4337-8ef9-b222b53a12da/0021e6ae-34c0-486e-ac47-c8566b803df5"
+					(reference "R81")
+					(unit 1)
+				)
+			)
+		)
+	)

Commit message: Fit the standard Ovonic 450 pack and recess the IO header
The earlier 50.5 x 25 x 14 mm pack size came from a mislabeled listing.
The layout now uses the standard Ovonic 80C 3S 450 mAh pack (design
envelope 46.5 x 25 x 21 mm) on top of the board, for a box of about
93.5 x 52 x 30 mm; the Long Size pack would have needed a ~110 mm box.

- S1-S6 (J5) move 5.55 mm inboard so the pin tips end 1 mm inside the
  left wall; the FET/shunt strip and nearby passives shift to suit.
- The pack carries a female XT30U-F, so J3 takes a male XT30U-M pigtail
  on 16 AWG. A vertical XT30UPB-M was checked and misses the 1 mm
  clearance under the face.
- IO1-IO4 GPIOs reordered for the new placement.

Schematic review passes; PCB review passes every gate except unrouted.

Co-Authored-By: Claude Opus 5.5 <noreply@anthropic.com>
Parts:
- J3: value XT30 pigtail 16AWG -> XT30U-M pigtail 16AWG
Changed lines of the file:
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@@
 			)
 		)
-		(property "Value" "XT30 pigtail 16AWG"
+		(property "Value" "XT30U-M pigtail 16AWG"
 			(at 153.67 172.72 0)
 			(show_name no)

Commit message: Use a vertical XT30 on the board instead of the pack pigtail
J3 is now an Amass XT30UPB-M (male, vertical, C428721) that the pack's
female XT30U-F plugs straight into; the pigtail pads and the reserved
mated-pair strip are removed and the pack power path re-routed.

The mated connector plus the 16 AWG bend needs 22.1-24.1 mm above the
board against 23.4 mm under the face of the 30 mm box. That is logged as
an enclosure open item to settle on the first prototype.

Schematic review passes; PCB review passes every gate except unrouted.

Co-Authored-By: Claude Opus 5.5 <noreply@anthropic.com>
Parts:
- J3: value XT30U-M pigtail 16AWG -> XT30UPB-M; footprint Connector_Wire:SolderWire-1.5sqmm_1x02_P6mm_D1.7mm_OD3mm -> hexy:AMASS_XT30UPB-M_1x02_P5.0mm_Vertical_EasyEDA3D; LCSC Part # (none) -> C428721; MPN (none) -> XT30UPB-M; Manufacturer (none) -> Changzhou Amass Elec
Changed lines of the file:
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@@
 			)
 		)
-		(property "Value" "XT30U-M pigtail 16AWG"
+		(property "Value" "XT30UPB-M"
 			(at 153.67 172.72 0)
 			(show_name no)
@@
 			)
 		)
-		(property "Footprint" "Connector_Wire:SolderWire-1.5sqmm_1x02_P6mm_D1.7mm_OD3mm"
+		(property "Footprint" "hexy:AMASS_XT30UPB-M_1x02_P5.0mm_Vertical_EasyEDA3D"
 			(at 160.02 170.18 0)
 			(hide yes)
@@
 			)
 		)
-		(property "MPN" ""
+		(property "MPN" "XT30UPB-M"
 			(at 160.02 170.18 0)
 			(effects
@@
 			)
 		)
-		(property "Manufacturer" ""
+		(property "Manufacturer" "Changzhou Amass Elec"
 			(at 160.02 170.18 0)
 			(effects
@@
 			)
 		)
+		(property "LCSC Part #" "C428721"
+			(at 160.02 172.72 0)
+			(hide yes)
+			(show_name no)
+			(do_not_autoplace no)
+			(effects
+				(font
+					(size 1.27 1.27)
+				)
+			)
+		)
